Commit message: Add Gazebo joint state bridge and update launch file for joint command bridging

File: mockway_moveit_servo/urdf/mockway_gazebo.urdf.xacro (robot description, xacro)
@@ -4,4 +4,11 @@
     <!-- Import the base mockway robot URDF -->
     <xacro:include filename="$(find mockway_description)/urdf/mockway_description.urdf" />
+    <!-- World link and fixed joint to ground the robot -->
+    <link name="world"/>
+    <joint name="world_to_base" type="fixed">
+        <parent link="world"/>
+        <child link="base_link"/>
+        <origin xyz="0 0 0" rpy="0 0 0"/>
+    </joint>
     <!-- Load initial positions -->
     <xacro:property name="initial_positions_file" value="$(arg initial_positions_file)" />
@@ -73,4 +80,55 @@
         </joint>
     </ros2_control>
+    <!-- Gazebo joint position controllers for each joint -->
+    <gazebo>
+        <plugin filename="gz-sim-joint-position-controller-system"
+                name="gz::sim::systems::JointPositionController">
+            <joint_name>joint1</joint_name>
+            <topic>/gz/mockway/joint1/cmd_pos</topic>
+            <p_gain>100</p_gain>
+            <i_gain>0.1</i_gain>
+            <d_gain>10</d_gain>
+        </plugin>
+        <plugin filename="gz-sim-joint-position-controller-system"
+                name="gz::sim::systems::JointPositionController">
+            <joint_name>joint2</joint_name>
+            <topic>/gz/mockway/joint2/cmd_pos</topic>
+            <p_gain>100</p_gain>
+            <i_gain>0.1</i_gain>
+            <d_gain>10</d_gain>
+        </plugin>
+        <plugin filename="gz-sim-joint-position-controller-system"
+                name="gz::sim::systems::JointPositionController">
+            <joint_name>joint3</joint_name>
+            <topic>/gz/mockway/joint3/cmd_pos</topic>
+            <p_gain>100</p_gain>
+            <i_gain>0.1</i_gain>
+            <d_gain>10</d_gain>
+        </plugin>
+        <plugin filename="gz-sim-joint-position-controller-system"
+                name="gz::sim::systems::JointPositionController">
+            <joint_name>joint4</joint_name>
+            <topic>/gz/mockway/joint4/cmd_pos</topic>
+            <p_gain>100</p_gain>
+            <i_gain>0.1</i_gain>
+            <d_gain>10</d_gain>
+        </plugin>
+        <plugin filename="gz-sim-joint-position-controller-system"
+                name="gz::sim::systems::JointPositionController">
+            <joint_name>joint5</joint_name>
+            <topic>/gz/mockway/joint5/cmd_pos</topic>
+            <p_gain>100</p_gain>
+            <i_gain>0.1</i_gain>
+            <d_gain>10</d_gain>
+        </plugin>
+        <plugin filename="gz-sim-joint-position-controller-system"
+                name="gz::sim::systems::JointPositionController">
+            <joint_name>joint6</joint_name>
+            <topic>/gz/mockway/joint6/cmd_pos</topic>
+            <p_gain>100</p_gain>
+            <i_gain>0.1</i_gain>
+            <d_gain>10</d_gain>
+        </plugin>
+    </gazebo>
     <!-- Gazebo material colors -->
     <gazebo reference="base_link">
