Commit message: 更新URDF

File: mockway_description/urdf/mockway_description.urdf (robot description, URDF)
Before this commit: robot mockway_description, 3 links, 2 joints
Links:
- added link link3, mass 0.481; collision mesh filename=package://mockway_description/meshes/link3.stl; visual mesh filename=package://mockway_description/meshes/link3.stl
- link link2: mass 0.915 -> 0.914
Joints:
- added joint joint3: type revolute, parent link2, child link3, origin xyz=0.000 0.190 0.000 rpy=0.000 -0.000 0.000, axis 0 0 1, limit lower=-3.140 upper=3.140 effort=9.000 velocity=3.140

Commit message: 装配体增加后盖，更新URDF

File: mockway_description/urdf/mockway_description.urdf (robot description, URDF)
Before this commit: robot mockway_description, 7 links, 6 joints
Links:
- link link1: mass 0.371 -> 0.378
- link link2: mass 0.914 -> 0.568
- link link3: mass 0.481 -> 0.488
- link link4: mass 0.371 -> 0.378
- link link5: mass 0.371 -> 0.378
