Commit message: feat(复现): 确保能复现仿真
- lua 运行时，分离npm install部分
- moveit 仿真部分确保use- 以及hardware:=true 工作正常
- 添加了 `Movelt2Ros.md` 以及 `Learn.md` 学习文档

File: moveit_mockway_config/config/mockway_description.ros2_control.xacro (robot description, xacro)
@@ -1,32 +1,12 @@
 <?xml version="1.0"?>
 <robot xmlns:xacro="http://www.ros.org/wiki/xacro">
-    <xacro:macro name="mockway_description_ros2_control" params="name initial_positions_file use_mock_hardware:=false">
+    <xacro:macro name="mockway_description_ros2_control" params="name initial_positions_file">
         <xacro:property name="initial_positions" value="${xacro.load_yaml(initial_positions_file)['initial_positions']}"/>
         <ros2_control name="${name}" type="system">
             <hardware>
-                <xacro:if value="${use_mock_hardware}">
-                    <!-- Mock hardware for simulation / testing -->
-                    <plugin>mock_components/GenericSystem</plugin>
-                </xacro:if>
-                <xacro:unless value="${use_mock_hardware}">
-                    <!-- DM Motor Hardware Interface for real hardware -->
-                    <plugin>dmmotor_hardware_interface/DMMototHardwareInterface</plugin>
-                    <!-- CAN interface configuration -->
-                    <!-- <param name="can_interface">can0</param> -->
-                    <param name="can_type">usb_can</param>
-                    <param name="can_interface">/dev/ttyUSB0</param>
-                    <param name="serial_baudrate">921600</param>
-                </xacro:unless>
+                <!-- By default, set up controllers for simulation. This won't work on real hardware -->
+                <plugin>mock_components/GenericSystem</plugin>
             </hardware>
-            <!-- Joint 1: DM-J4310-2EC -->
             <joint name="joint1">
-                <param name="can_id">0x01</param>
-                <param name="kp">50.0</param>
-                <param name="kd">1.0</param>
-                <!-- type: 1 DM4310, 2 DM4310_48V, 3 DM4340, 4 DM4340_48V -->
-                <param name="type">1</param>
-                <!-- dir: 1 pos, -1 neg -->
-                <param name="dir">1</param>
-                <param name="is_simulated">false</param>
                 <command_interface name="position"/>
                 <state_interface name="position">
@@ -35,12 +15,5 @@
                 <state_interface name="velocity"/>
             </joint>
-            <!-- Joint 2: DM4340 -->
             <joint name="joint2">
-                <param name="can_id">0x02</param>
-                <param name="kp">500.0</param>
-                <param name="kd">3.0</param>
-                <param name="type">3</param>
-                <param name="dir">1</param>
-                <param name="is_simulated">false</param>
                 <command_interface name="position"/>
                 <state_interface name="position">
@@ -49,12 +22,5 @@
                 <state_interface name="velocity"/>
             </joint>
-            <!-- Joint 3: DM4340 -->
             <joint name="joint3">
-                <param name="can_id">0x03</param>
-                <param name="kp">450.0</param>
-                <param name="kd">2.0</param>
-                <param name="type">3</param>
-                <param name="dir">-1</param>
-                <param name="is_simulated">false</param>
                 <command_interface name="position"/>
                 <state_interface name="position">
@@ -63,12 +29,5 @@
                 <state_interface name="velocity"/>
             </joint>
-            <!-- Joint 4: DM-J4310-2EC -->
             <joint name="joint4">
-                <param name="can_id">0x04</param>
-                <param name="kp">90.0</param>
-                <param name="kd">1.0</param>
-                <param name="type">1</param>
-                <param name="dir">1</param>
-                <param name="is_simulated">false</param>
                 <command_interface name="position"/>
                 <state_interface name="position">
@@ -77,12 +36,5 @@
                 <state_interface name="velocity"/>
             </joint>
-            <!-- Joint 5: DM-J4310-2EC -->
             <joint name="joint5">
-                <param name="can_id">0x05</param>
-                <param name="kp">50.0</param>
-                <param name="kd">0.8</param>
-                <param name="type">1</param>
-                <param name="dir">1</param>
-                <param name="is_simulated">false</param>
                 <command_interface name="position"/>
                 <state_interface name="position">
@@ -91,12 +43,5 @@
                 <state_interface name="velocity"/>
             </joint>
-            <!-- Joint 6: DM-J4310-2EC -->
             <joint name="joint6">
-                <param name="can_id">0x06</param>
-                <param name="kp">50.0</param>
-                <param name="kd">0.8</param>
-                <param name="type">1</param>
-                <param name="dir">1</param>
-                <param name="is_simulated">false</param>
                 <command_interface name="position"/>
                 <state_interface name="position">

File: moveit_mockway_config/config/mockway_description.urdf.xacro (robot description, xacro)
@@ -2,9 +2,8 @@
 <robot xmlns:xacro="http://www.ros.org/wiki/xacro" name="mockway_description">
     <xacro:arg name="initial_positions_file" default="initial_positions.yaml" />
-    <xacro:arg name="use_mock_hardware" default="false" />
     <!-- Import mockway_description urdf file -->
     <xacro:include filename="$(find mockway_description)/urdf/mockway_description.urdf" />
     <!-- Import control_xacro -->
     <xacro:include filename="mockway_description.ros2_control.xacro" />
-    <xacro:mockway_description_ros2_control name="MockwaySystem" initial_positions_file="$(arg initial_positions_file)" use_mock_hardware="$(arg use_mock_hardware)"/>
+    <xacro:mockway_description_ros2_control name="FakeSystem" initial_positions_file="$(arg initial_positions_file)"/>
 </robot>

Commit message: feat(gazebo): support gazebo simulation

File: moveit_mockway_config/config/mockway_description.ros2_control.xacro (robot description, xacro)
@@ -1,10 +1,16 @@
 <?xml version="1.0"?>
 <robot xmlns:xacro="http://www.ros.org/wiki/xacro">
-    <xacro:macro name="mockway_description_ros2_control" params="name initial_positions_file">
+    <xacro:macro name="mockway_description_ros2_control" params="name initial_positions_file use_gazebo:=false">
         <xacro:property name="initial_positions" value="${xacro.load_yaml(initial_positions_file)['initial_positions']}"/>
         <ros2_control name="${name}" type="system">
             <hardware>
-                <!-- By default, set up controllers for simulation. This won't work on real hardware -->
-                <plugin>mock_components/GenericSystem</plugin>
+                <!-- gazebo simulation -->
+                <xacro:if value="${use_gazebo}">
+                    <plugin>gz_ros2_control/GazeboSimSystem</plugin>
+                </xacro:if>
+                <xacro:unless value="${use_gazebo}">
+                    <!-- By default, set up controllers for simulation. This won't work on real hardware -->
+                    <plugin>mock_components/GenericSystem</plugin>
+                </xacro:unless>
             </hardware>
             <joint name="joint1">

File: moveit_mockway_config/config/mockway_description.urdf.xacro (robot description, xacro)
@@ -2,8 +2,26 @@
 <robot xmlns:xacro="http://www.ros.org/wiki/xacro" name="mockway_description">
     <xacro:arg name="initial_positions_file" default="initial_positions.yaml" />
+    <!-- If gazebo -->
+    <xacro:arg name="use_gazebo" default="false" />
     <!-- Import mockway_description urdf file -->
     <xacro:include filename="$(find mockway_description)/urdf/mockway_description.urdf" />
     <!-- Import control_xacro -->
     <xacro:include filename="mockway_description.ros2_control.xacro" />
-    <xacro:mockway_description_ros2_control name="FakeSystem" initial_positions_file="$(arg initial_positions_file)"/>
+    <xacro:mockway_description_ros2_control name="FakeSystem" initial_positions_file="$(arg initial_positions_file)" use_gazebo="$(arg use_gazebo)"/>
+    <xacro:if value="$(arg use_gazebo)">
+        <!-- Gazebo 中固定底座，防止 base_link 作为自由刚体受重力掉落或倾倒。 -->
+        <link name="world"/>
+        <joint name="world_fixed" type="fixed">
+            <parent link="world"/>
+            <child link="base_link"/>
+            <origin xyz="0 0 0.02" rpy="0 0 0"/>
+        </joint>
+        <gazebo>
+            <plugin filename="gz_ros2_control-system" name="gz_ros2_control::GazeboSimROS2ControlPlugin">
+                <parameters>
+                    $(find moveit_mockway_config)/config/ros2_controllers.yaml
+                </parameters>
+            </plugin>
+        </gazebo>
+    </xacro:if>
 </robot>
